Commit message: finished but not tested hoverboard driver

File: src/robot_description/src/description/robot_description.urdf (robot description, URDF)
Before this commit: robot robot, 7 links, 6 joints
Links:
- removed link camera_depth_frame
- removed link camera_link
Joints:
- removed joint camera_depth_joint
- removed joint camera_joint
